Commit message: Edit collision geometry

File: bbot_description/urdf/bbot.urdf.xacro (robot description, xacro)
@@ -10,7 +10,9 @@
     <link name="main_base">
       <inertial>
-        <origin xyz="0.023151 -0.0 0.069877" />
+        <!-- <origin xyz="0.023151 -0.0 0.069877" /> OLD -->
+        <origin xyz="0.02228462 0.05671578 -0.01906787" rpy="0.0 0 0" />
         <mass value="1.171185"/>
-        <inertia ixx="1.0" ixy="0.0" ixz="0.0" iyy="1.0" iyz="0.0" izz="1.0" />
+        <!-- <inertia ixx="1.0" ixy="0.0" ixz="0.0" iyy="1.0" iyz="0.0" izz="1.0" /> OLD -->
+        <inertia ixx="0.00249622" ixy="0.00000872" ixz="-0.00002689" iyy="0.00361734" iyz="-0.00004823" izz="0.00381216" />
       </inertial>
       <visual>
@@ -21,7 +23,8 @@
       </visual>
       <collision>
-        <origin xyz="0.0 0.0 0.0" rpy="1.57 0 0" />
-        <geometry>
-          <mesh filename="package://bbot_description/meshes/collision/base.stl"  scale="1 1 1"/>
+        <origin xyz="0.023030 0.017698 0.066007" rpy="0.0 0 0" />
+        <geometry>
+          <!-- <mesh filename="package://bbot_description/meshes/collision/base.stl"  scale="1 1 1"/> -->
+          <box size="0.174214 0.139588 0.096376" />
         </geometry>
       </collision>
@@ -40,7 +43,9 @@
       </visual>
       <collision>
-        <origin xyz="-0.025 -0.021 -0.18" rpy="-1.57 -1.57 0" />
-        <geometry>
-          <mesh filename="package://bbot_description/meshes/collision/right_top_leg.stl"  scale="1 1 1"/>
+        <!-- <origin xyz="-0.025 -0.021 -0.18" rpy="-1.57 -1.57 0" /> MESH ORIGIN -->
+        <origin xyz="0.031 0 -0.055" rpy="0 0 0" />
+        <geometry>
+          <!-- <mesh filename="package://bbot_description/meshes/collision/right_top_leg.stl"  scale="1 1 1"/> -->
+           <box size="0.065065 0.048933 0.138999" />
         </geometry>
       </collision>
@@ -59,7 +64,9 @@
       </visual>
       <collision>
-        <origin xyz="-0.031 -0.021 -0.19" rpy="-1.57 -1.57 0" />
-        <geometry>
-          <mesh filename="package://bbot_description/meshes/collision/left_top_leg.stl"  scale="1 1 1"/>
+        <!-- <origin xyz="-0.031 -0.021 -0.19" rpy="-1.57 -1.57 0" /> MESH ORIGIN -->
+        <origin xyz="-0.031 0 -0.055" rpy="0 0 0" />
+        <geometry>
+          <!-- <mesh filename="package://bbot_description/meshes/collision/left_top_leg.stl"  scale="1 1 1"/> -->
+          <box size="0.065065 0.048933 0.138999" />
         </geometry>
       </collision>
@@ -78,7 +85,9 @@
       </visual>
       <collision>
-        <origin xyz="-0.025 -0.021 -0.0695" rpy="-1.57 -1.57 0" />
-        <geometry>
-          <mesh filename="package://bbot_description/meshes/collision/right_bottom_leg.stl"  scale="1 1 1"/>
+        <!-- <origin xyz="-0.025 -0.021 -0.0695" rpy="-1.57 -1.57 0" />  MESH ORIGIN-->
+        <origin xyz="0.02825 0 -0.065" rpy="0 0 0" />
+        <geometry>
+          <!-- <mesh filename="package://bbot_description/meshes/collision/right_bottom_leg.stl"  scale="1 1 1"/> -->
+          <box size="0.040031 0.054258 0.071798" />
         </geometry>
       </collision>
@@ -97,7 +106,9 @@
       </visual>
       <collision>
-        <origin xyz="-0.031 -0.021 -0.0795" rpy="-1.57 -1.57 0" />
-        <geometry>
-          <mesh filename="package://bbot_description/meshes/collision/left_bottom_leg.stl"  scale="1 1 1"/>
+        <!-- <origin xyz="-0.031 -0.021 -0.0795" rpy="-1.57 -1.57 0" /> MESH ORIGIN -->
+        <origin xyz="-0.02825 0 -0.065" rpy="0 0 0" />
+        <geometry>
+          <!-- <mesh filename="package://bbot_description/meshes/collision/left_bottom_leg.stl"  scale="1 1 1"/> -->
+          <box size="0.040031 0.054258 0.071798" />
         </geometry>
       </collision>
@@ -105,5 +116,5 @@
     <link name="right_wheel">
       <inertial>
-        <origin xyz="0 0 0" />
+       <origin xyz="0 0 0" />
         <mass value="0.303077"/>
         <inertia ixx="1.0" ixy="0.0" ixz="0.0" iyy="1.0" iyz="0.0" izz="1.0" />
@@ -116,7 +127,9 @@
       </visual>
       <collision>
-        <origin xyz="-0.019 0.009 0.021" rpy="0 0 1.57" />
-        <geometry>
-          <mesh filename="package://bbot_description/meshes/collision/right_wheel.stl"  scale="1 1 1"/>
+        <!-- <origin xyz="-0.019 0.009 0.021" rpy="0 0 1.57" /> MESH ORIGIN -->
+        <origin xyz="-0.002 -0.0003 0" rpy="1.57 0 1.57" />
+        <geometry>
+          <!-- <mesh filename="package://bbot_description/meshes/collision/right_wheel.stl"  scale="1 1 1"/> -->
+          <cylinder radius="0.05" length="0.03"/>
         </geometry>
       </collision>
@@ -135,7 +148,9 @@
       </visual>
       <collision>
-        <origin xyz="-0.037 0.0 -0.021" rpy="0 0 -1.57" />
-        <geometry>
-          <mesh filename="package://bbot_description/meshes/collision/left_wheel.stl"  scale="1 1 1"/>
+        <!-- <origin xyz="-0.037 0.0 -0.021" rpy="0 0 -1.57" /> MESH ORIGIN -->
+        <origin xyz="0.0015 -0.0003 0" rpy="1.57 0 1.57" />
+        <geometry>
+          <!-- <mesh filename="package://bbot_description/meshes/collision/left_wheel.stl"  scale="1 1 1"/> -->
+          <cylinder radius="0.05" length="0.03"/>
         </geometry>
       </collision>
@@ -154,7 +169,9 @@
       </visual>
       <collision>
-        <origin xyz="-0.0 -0.0 0.0" rpy="-1.57 -1.57 0" />
-        <geometry>
-          <mesh filename="package://bbot_description/meshes/collision/LDS.stl"  scale="1 1 1"/>
+        <!-- <origin xyz="0.022746 0.022746 0.137604" rpy="-1.57 -1.57 0" /> MESH ORIGIN -->
+        <origin xyz=" -0.02 0.0 0.025" rpy="1.57 0 0" />
+        <geometry>
+          <!-- <mesh filename="package://bbot_description/meshes/collision/LDS.stl"  scale="1 1 1"/> -->
+          <box size="0.069747 0.103263 0.038782" />
         </geometry>
       </collision>
@@ -175,5 +192,6 @@
         <origin xyz="-0.0 -0.0 0.0" rpy="0 0 0" />
         <geometry>
-          <mesh filename="package://bbot_description/meshes/collision/RspCameraV2.stl"  scale="1 1 1"/>
+          <!-- <mesh filename="package://bbot_description/meshes/collision/RspCameraV2.stl"  scale="1 1 1"/> -->
+          <box size="0.001 0.001 0.001"/>
         </geometry>
       </collision>

Commit message: Correct inertial features

File: bbot_description/urdf/bbot.urdf.xacro (robot description, xacro)
@@ -10,9 +10,7 @@
     <link name="main_base">
       <inertial>
-        <!-- <origin xyz="0.023151 -0.0 0.069877" /> OLD -->
-        <origin xyz="0.02228462 0.05671578 -0.01906787" rpy="0.0 0 0" />
+        <origin xyz="0.02228462 0.01906787 0.05671578" rpy="0.0 0 0" />
         <mass value="1.171185"/>
-        <!-- <inertia ixx="1.0" ixy="0.0" ixz="0.0" iyy="1.0" iyz="0.0" izz="1.0" /> OLD -->
-        <inertia ixx="0.00249622" ixy="0.00000872" ixz="-0.00002689" iyy="0.00361734" iyz="-0.00004823" izz="0.00381216" />
+        <inertia ixx="0.00249108" ixy="0.0" ixz="0.0" iyy="0.0038043" iyz="0.0" izz="0.00360989" />
       </inertial>
       <visual>
@@ -34,5 +32,5 @@
         <origin xyz="0.032 0 -0.072" />
         <mass value="0.237123"/>
-        <inertia ixx="1.0" ixy="0.0" ixz="0.0" iyy="1.0" iyz="0.0" izz="1.0" />
+        <inertia ixx="0.00025778" ixy="0.0" ixz="0.0" iyy="0.00029723" iyz="0.0" izz="0.00010339" />
       </inertial>
       <visual>
@@ -55,5 +53,5 @@
         <origin xyz="-0.032 0 -0.072" />
         <mass value="0.237123"/>
-        <inertia ixx="1.0" ixy="0.0" ixz="0.0" iyy="1.0" iyz="0.0" izz="1.0" />
+        <inertia ixx="0.00025778" ixy="0.0" ixz="0.0" iyy="0.00029723" iyz="0.0" izz="0.00010339" />
       </inertial>
       <visual>
@@ -76,5 +74,5 @@
         <origin xyz="0.032 0 -0.06525" />
         <mass value="0.367745"/>
-        <inertia ixx="1.0" ixy="0.0" ixz="0.0" iyy="1.0" iyz="0.0" izz="1.0" />
+        <inertia ixx="0.00034532" ixy="0.0" ixz="-0.00001256" iyy="0.00035624" iyz="0.0" izz="0.00016337" />
       </inertial>
       <visual>
@@ -97,5 +95,5 @@
         <origin xyz="-0.032 0 -0.06525" />
         <mass value="0.367745"/>
-        <inertia ixx="1.0" ixy="0.0" ixz="0.0" iyy="1.0" iyz="0.0" izz="1.0" />
+        <inertia ixx="0.00034531" ixy="0.0" ixz="-0.00001256" iyy="0.00035624" iyz="0.0" izz="0.00016337" />
       </inertial>
       <visual>
@@ -116,7 +114,7 @@
     <link name="right_wheel">
       <inertial>
-       <origin xyz="0 0 0" />
+        <origin xyz="0 0 0" />
         <mass value="0.303077"/>
-        <inertia ixx="1.0" ixy="0.0" ixz="0.0" iyy="1.0" iyz="0.0" izz="1.0" />
+        <inertia ixx="0.00038173" ixy="0.0" ixz="0.0" iyy="0.00021305" iyz="0.0" izz="0.00021285" />
       </inertial>
       <visual>
@@ -139,5 +137,5 @@
         <origin xyz="0 0 0"/>
         <mass value="0.303077"/>
-        <inertia ixx="1.0" ixy="0.0" ixz="0.0" iyy="1.0" iyz="0.0" izz="1.0" />
+        <inertia ixx="0.00038173" ixy="0.0" ixz="0.0" iyy="0.00021305" iyz="0.0" izz="0.00021285" />
       </inertial>
       <visual>
@@ -160,5 +158,5 @@
         <origin xyz="0 0 0" />
         <mass value="0.125"/>
-        <inertia ixx="1.0" ixy="0.0" ixz="0.0" iyy="1.0" iyz="0.0" izz="1.0" />
+        <inertia ixx="0.00005831" ixy="0.0" ixz="0.0" iyy="0.00006409" iyz="0.0" izz="0.00011932" />
       </inertial>
       <visual>
@@ -181,5 +179,5 @@
         <origin xyz="0 0 0" />
         <mass value="0.003"/>
-        <inertia ixx="1.0" ixy="0.0" ixz="0.0" iyy="1.0" iyz="0.0" izz="1.0" />
+        <inertia ixx="1.4e-7" ixy="0.0" ixz="0.0" iyy="2.4e-7" iyz="0.0" izz="1.2e-7" />
       </inertial>
       <visual>

Commit message: Update IMU data

File: bbot_description/urdf/bbot.urdf.xacro (robot description, xacro)
@@ -448,5 +448,31 @@
     </gazebo>
   <!-- IMU -->
-    <gazebo>
+    <link name="imu_frame_gazebo"/>
+    <joint name="imu_joint" type="fixed">
+        <parent link="main_base" />
+        <child link="imu_frame_gazebo" />
+        <origin xyz="0.02075 0.01765 0.0326" rpy="0 0 0" />
+    </joint>
+    <gazebo reference="imu_frame_gazebo">
+      <gravity>true</gravity>
+      <sensor name="imu_sensor" type="imu">
+        <always_on>true</always_on>
+        <update_rate>100</update_rate>
+        <visualize>true</visualize>
+        <pose>0 0 0 0 0 0</pose>
+        <topic>__default_topic__</topic>
+        <plugin filename="libgazebo_ros_imu_sensor.so" name="imu_plugin">
+          <topicName>/bbot/imu</topicName>
+          <bodyName>imu_frame_gazebo</bodyName>
+          <updateRateHZ>10.0</updateRateHZ>
+          <gaussianNoise>0.0</gaussianNoise>
+          <xyzOffset>0 0 0</xyzOffset>
+          <rpyOffset>0 0 0</rpyOffset>
+          <frameName>imu_frame_gazebo</frameName>
+          <initialOrientationAsReference>false</initialOrientationAsReference>
+        </plugin>
+      </sensor>
+    </gazebo>
+    <!-- <gazebo reference="imu_frame_gazebo">
       <plugin filename="libgazebo_ros_imu.so" name="imu_plugin">
         <alwaysOn>true</alwaysOn>
@@ -459,4 +485,4 @@
         <rpyOffset>0 0 0</rpyOffset>
       </plugin>
-    </gazebo>
+    </gazebo>  -->
 </robot>

Commit message: Fix TF issues and increase imu freq

File: bbot_description/urdf/bbot.urdf.xacro (robot description, xacro)
@@ -6,4 +6,5 @@
     <parent link="base_link"/>
     <child link="main_base"/>
+    <origin xyz="0.0 0.0 0.0" rpy="0.0 0.0 1.57" />
   </joint>
 <!-- LINKS -->
@@ -465,5 +466,5 @@
           <topicName>/bbot/imu</topicName>
           <bodyName>imu_frame_gazebo</bodyName>
-          <updateRateHZ>10.0</updateRateHZ>
+          <updateRateHZ>100.0</updateRateHZ>
           <gaussianNoise>0.0</gaussianNoise>
           <xyzOffset>0 0 0</xyzOffset>

Commit message: modificando meshes do robo

File: bbot_description/urdf/bbot.urdf.xacro (robot description, xacro)
@@ -78,5 +78,5 @@
       </inertial>
       <visual>
-        <origin xyz="-0.025 -0.021 -0.0695" rpy="-1.57 -1.57 0" />
+        <origin xyz="0.0275 0.027 -0.06386394" rpy="-1.57 -1.57 0" />
         <geometry>
           <mesh filename="package://bbot_description/meshes/visual/right_bottom_leg.dae"  scale="1 1 1"/>
@@ -85,5 +85,5 @@
       <collision>
         <!-- <origin xyz="-0.025 -0.021 -0.0695" rpy="-1.57 -1.57 0" />  MESH ORIGIN-->
-        <origin xyz="0.02825 0 -0.065" rpy="0 0 0" />
+        <origin xyz="0.03013079 0 -0.065" rpy="0 0 0" />
         <geometry>
           <!-- <mesh filename="package://bbot_description/meshes/collision/right_bottom_leg.stl"  scale="1 1 1"/> -->
@@ -99,5 +99,5 @@
       </inertial>
       <visual>
-        <origin xyz="-0.031 -0.021 -0.0795" rpy="-1.57 -1.57 0" />
+        <origin xyz="-0.0292 0.027 -0.06867645" rpy="1.57 -1.57 0" />
         <geometry>
           <mesh filename="package://bbot_description/meshes/visual/left_bottom_leg.dae"  scale="1 1 1"/>
@@ -162,5 +162,5 @@
       </inertial>
       <visual>
-        <origin xyz="-0.0 -0.0 0.0" rpy="-1.57 -1.57 0" />
+        <origin xyz="0.0 0.01 0.0" rpy="-1.57 -1.57 0" />
         <geometry>
           <mesh filename="package://bbot_description/meshes/visual/LDS.dae"  scale="1 1 1"/>
@@ -183,5 +183,5 @@
       </inertial>
       <visual>
-        <origin xyz="-0.0 -0.0 0.0" rpy="0 0 0" />
+        <origin xyz="0.0 0.0 0.01" rpy="0 0 0" />
         <geometry>
           <mesh filename="package://bbot_description/meshes/visual/RspCameraV2.dae"  scale="1 1 1"/>

Commit message: Update mass and inertial features of the legs and wheels

File: bbot_description/urdf/bbot.urdf.xacro (robot description, xacro)
@@ -1,4 +1,6 @@
 <?xml version="1.0" ?>
 <robot name="Bbot" xmlns:xacro="http://www.ros.org/wiki/xacro">
+<!-- INFO -->
+<!-- Center of Mass height: 0.235 m -->
 <!-- Dummy Root Link -->
   <link name="base_link"/>
@@ -13,5 +15,5 @@
         <origin xyz="0.02228462 0.01906787 0.05671578" rpy="0.0 0 0" />
         <mass value="1.171185"/>
-        <inertia ixx="0.00249108" ixy="0.0" ixz="0.0" iyy="0.0038043" iyz="0.0" izz="0.00360989" />
+        <inertia ixx="0.00311204" ixy="0.0" ixz="0.0" iyy="0.00402789" iyz="0.0" izz="0.00411583" />
       </inertial>
       <visual>
@@ -32,6 +34,6 @@
       <inertial>
         <origin xyz="0.032 0 -0.072" />
-        <mass value="0.237123"/>
-        <inertia ixx="0.00025778" ixy="0.0" ixz="0.0" iyy="0.00029723" iyz="0.0" izz="0.00010339" />
+        <mass value="0.207"/>
+        <inertia ixx="0.00022502" ixy="0.0" ixz="0.0" iyy="0.00025945" iyz="0.0" izz="0.00009025" />
       </inertial>
       <visual>
@@ -53,6 +55,6 @@
       <inertial>
         <origin xyz="-0.032 0 -0.072" />
-        <mass value="0.237123"/>
-        <inertia ixx="0.00025778" ixy="0.0" ixz="0.0" iyy="0.00029723" iyz="0.0" izz="0.00010339" />
+        <mass value="0.207"/>
+        <inertia ixx="0.00022502" ixy="0.0" ixz="0.0" iyy="0.00025945" iyz="0.0" izz="0.00009025" />
       </inertial>
       <visual>
@@ -74,6 +76,6 @@
       <inertial>
         <origin xyz="0.032 0 -0.06525" />
-        <mass value="0.367745"/>
-        <inertia ixx="0.00034532" ixy="0.0" ixz="-0.00001256" iyy="0.00035624" iyz="0.0" izz="0.00016337" />
+        <mass value="0.334"/>
+        <inertia ixx="0.0003166" ixy="0.0" ixz="0.0" iyy="0.00032649" iyz="0.0" izz="0.00014826" />
       </inertial>
       <visual>
@@ -95,6 +97,6 @@
       <inertial>
         <origin xyz="-0.032 0 -0.06525" />
-        <mass value="0.367745"/>
-        <inertia ixx="0.00034531" ixy="0.0" ixz="-0.00001256" iyy="0.00035624" iyz="0.0" izz="0.00016337" />
+        <mass value="0.334"/>
+        <inertia ixx="0.0003166" ixy="0.0" ixz="0.0" iyy="0.00032649" iyz="0.0" izz="0.00014826" />
       </inertial>
       <visual>
@@ -117,5 +119,5 @@
         <origin xyz="0 0 0" />
         <mass value="0.303077"/>
-        <inertia ixx="0.00038173" ixy="0.0" ixz="0.0" iyy="0.00021305" iyz="0.0" izz="0.00021285" />
+        <inertia ixx="0.0002521" ixy="0.0" ixz="0.0" iyy="0.00014179" iyz="0.0" izz="0.00014098" />
       </inertial>
       <visual>
@@ -138,5 +140,5 @@
         <origin xyz="0 0 0"/>
         <mass value="0.303077"/>
-        <inertia ixx="0.00038173" ixy="0.0" ixz="0.0" iyy="0.00021305" iyz="0.0" izz="0.00021285" />
+        <inertia ixx="0.0002521" ixy="0.0" ixz="0.0" iyy="0.00014179" iyz="0.0" izz="0.00014098" />
       </inertial>
       <visual>

Commit message: Add balancing PID node. Update configs and README

File: bbot_description/urdf/bbot.urdf.xacro (robot description, xacro)
@@ -3,4 +3,8 @@
 <!-- INFO -->
 <!-- Center of Mass height: 0.235 m -->
+<!-- Top leg lengh: 0.1106 m -->
+<!-- Bottom leg lengh: 0.0795 m -->
+<!-- Max alpha: 46º -->
+<!-- Max Betha: 140º -->
 <!-- Dummy Root Link -->
   <link name="base_link"/>
@@ -27,5 +31,5 @@
         <geometry>
           <!-- <mesh filename="package://bbot_description/meshes/collision/base.stl"  scale="1 1 1"/> -->
-          <box size="0.174214 0.139588 0.096376" />
+          <box size="0.174214 0.159979 0.096376" />
         </geometry>
       </collision>
@@ -122,5 +126,5 @@
       </inertial>
       <visual>
-        <origin xyz="-0.019 0.009 0.021" rpy="0 0 1.57" />
+        <origin xyz="-0.019 0.0095 0.021" rpy="0 0 1.57" />
         <geometry>
           <mesh filename="package://bbot_description/meshes/visual/right_wheel.dae"  scale="1 1 1"/>
@@ -150,5 +154,5 @@
       <collision>
         <!-- <origin xyz="-0.037 0.0 -0.021" rpy="0 0 -1.57" /> MESH ORIGIN -->
-        <origin xyz="0.0015 -0.0003 0" rpy="1.57 0 1.57" />
+        <origin xyz="0.002 -0.0003 0" rpy="1.57 0 1.57" />
         <geometry>
           <!-- <mesh filename="package://bbot_description/meshes/collision/left_wheel.stl"  scale="1 1 1"/> -->
@@ -202,5 +206,5 @@
       <parent link="main_base"/>
       <child link="right_top_leg"/>
-      <origin xyz="-0.055 0.021 0.0" rpy="0 0 0" />
+      <origin xyz="-0.055 0.021 0.0" rpy="0.656 0 0" /> <!-- Previous 0.656 0.3927 -->
       <axis xyz="1 0 0" />
       <limit velocity="6.5" effort="1000" lower="-3.14" upper="3.14" />
@@ -210,5 +214,5 @@
       <parent link="main_base"/>
       <child link="left_top_leg"/>
-      <origin xyz="0.101 0.021 0.0" rpy="0 0 0" />
+      <origin xyz="0.101 0.021 0.0" rpy="0.656 0 0" />
       <axis xyz="1 0 0" />
       <limit velocity="6.5" effort="1000" lower="-3.14" upper="3.14" />
@@ -218,5 +222,5 @@
       <parent link="right_top_leg"/>
       <child link="right_bottom_leg"/>
-      <origin xyz="-0.0 0.0 -0.1105" rpy="0 0 0" />
+      <origin xyz="-0.0 0.0 -0.1105" rpy="-1.67 0 0" /> <!-- Previous -1.67 -0.9547-->
       <axis xyz="1 0 0" />
       <limit velocity="6.5" effort="1000" lower="-3.14" upper="3.14" />
@@ -226,24 +230,24 @@
       <parent link="left_top_leg"/>
       <child link="left_bottom_leg"/>
-      <origin xyz="-0.0 0.0 -0.1105" rpy="0 0 0" />
+      <origin xyz="-0.0 0.0 -0.1105" rpy="-1.67 0 0" />
       <axis xyz="1 0 0" />
       <limit velocity="6.5" effort="1000" lower="-3.14" upper="3.14" />
       <dynamics damping="0.1" friction="0.0" />
     </joint>
-    <joint name="right_bottom_leg2wheel" type="revolute">
+    <joint name="right_bottom_leg2wheel" type="continuous">
       <parent link="right_bottom_leg"/>
       <child link="right_wheel"/>
       <origin xyz="-0.0062 0.0 -0.0795" rpy="0 0 0" />
       <axis xyz="1 0 0" />
-      <limit velocity="500" effort="1000" lower="-2.0944" upper="2.0944" />
-      <dynamics damping="0.1" friction="0.0" />
-    </joint>
-    <joint name="left_bottom_leg2wheel" type="revolute">
+      <limit velocity="500" effort="1000"/> <!--lower="-2.0944" upper="2.0944"-->
+      <dynamics damping="0.01" friction="0.0" />
+    </joint>
+    <joint name="left_bottom_leg2wheel" type="continuous">
       <parent link="left_bottom_leg"/>
       <child link="left_wheel"/>
       <origin xyz="0.0062 0.0 -0.0795" rpy="0 0 0" />
       <axis xyz="1 0 0" />
-      <limit velocity="500" effort="1000" lower="-2.0944" upper="2.0944" />
-      <dynamics damping="0.1" friction="0.0" />
+      <limit velocity="500" effort="1000"/> <!--lower="-2.0944" upper="2.0944"-->
+      <dynamics damping="0.01" friction="0.0" />
     </joint>
     <joint name="base2lds" type="fixed">
@@ -325,38 +329,38 @@
 <!-- PARAMETERS -->
   <gazebo reference="main_base">
-      <mu1>0.2</mu1>
-      <mu2>0.2</mu2>
+      <mu1>0.5</mu1>
+      <mu2>0.5</mu2>
   </gazebo>
   <gazebo reference="right_top_leg">
-      <mu1>0.2</mu1>
-      <mu2>0.2</mu2>
+      <mu1>0.5</mu1>
+      <mu2>0.5</mu2>
   </gazebo>
   <gazebo reference="left_top_leg">
-      <mu1>0.2</mu1>
-      <mu2>0.2</mu2>
+      <mu1>0.5</mu1>
+      <mu2>0.5</mu2>
   </gazebo>
   <gazebo reference="right_bottom_leg">
-      <mu1>0.2</mu1>
-      <mu2>0.2</mu2>
+      <mu1>0.5</mu1>
+      <mu2>0.5</mu2>
   </gazebo>
   <gazebo reference="left_bottom_leg">
-      <mu1>0.2</mu1>
-      <mu2>0.2</mu2>
+      <mu1>0.5</mu1>
+      <mu2>0.5</mu2>
   </gazebo>
   <gazebo reference="right_wheel">
-      <mu1>0.2</mu1>
-      <mu2>0.2</mu2>
+      <mu1>0.8</mu1>
+      <mu2>0.8</mu2>
   </gazebo>
   <gazebo reference="left_wheel">
-      <mu1>0.2</mu1>
-      <mu2>0.2</mu2>
+      <mu1>0.8</mu1>
+      <mu2>0.8</mu2>
   </gazebo>
   <gazebo reference="lds">
-      <mu1>0.2</mu1>
-      <mu2>0.2</mu2>
+      <mu1>0.5</mu1>
+      <mu2>0.5</mu2>
   </gazebo>
   <gazebo reference="RspCameraV2">
-      <mu1>0.2</mu1>
-      <mu2>0.2</mu2>
+      <mu1>0.5</mu1>
+      <mu2>0.5</mu2>
   </gazebo>
 <!-- SENSOR -->
@@ -456,4 +460,5 @@
         <child link="imu_frame_gazebo" />
         <origin xyz="0.02075 0.01765 0.0326" rpy="0 0 0" />
+        <!-- <origin xyz="-0.01765 0.02075 0.0326" rpy="0 0 0" /> -->
     </joint>
     <gazebo reference="imu_frame_gazebo">
