Commit message: Add tag detection

File: bbot_description/urdf/bbot.urdf.xacro (robot description, xacro)
@@ -189,5 +189,5 @@
       </inertial>
       <visual>
-        <origin xyz="0.0 0.0 0.01" rpy="0 0 0" />
+        <origin xyz="0.023 0.036 -0.15" rpy="0 0 -1.57" />
         <geometry>
           <mesh filename="package://bbot_description/meshes/visual/RspCameraV2.dae"  scale="1 1 1"/>
@@ -259,5 +259,5 @@
       <parent link="main_base"/>
       <child link="RspCameraV2"/>
-      <origin xyz="0.0 0.13 0.0" rpy="1.57 -1.57 0" />
+      <origin xyz="0.023 -0.03 0.036" rpy="1.57 3.14 0" />
     </joint>
 <!-- TRANSMISSION -->
@@ -370,5 +370,5 @@
         <parent link="RspCameraV2" />
         <child link="camera_frame_gazebo" />
-        <origin xyz="0.036 -0.023 0.16" rpy="1.57 -1.57 1.57" />
+        <origin xyz="0 0 0" rpy="1.57 -1.57 0" />
     </joint>
     <gazebo reference="camera_frame_gazebo">
@@ -426,5 +426,5 @@
       <sensor type="gpu_ray" name="lds_sensor">
         <pose>0 0 0 0 0 0</pose>
-        <visualize>false</visualize>
+        <visualize>true</visualize>
         <update_rate>40</update_rate>
         <ray>
@@ -439,5 +439,5 @@
           <range>
             <min>0.12</min>
-            <max>3.5</max>
+            <max>1.2</max>
             <resolution>0.01</resolution>
           </range>
@@ -450,5 +450,5 @@
         <plugin name="gazebo_ros_head_hokuyo_controller" filename="libgazebo_ros_gpu_laser.so">
           <topicName>/bbot/laser/scan</topicName>
-          <frameName>odom</frameName>
+          <frameName>lds_frame_gazebo</frameName>
         </plugin>
       </sensor>

Commit message: Add leg controllers

File: bbot_description/urdf/bbot.urdf.xacro (robot description, xacro)
@@ -206,5 +206,5 @@
       <parent link="main_base"/>
       <child link="right_top_leg"/>
-      <origin xyz="-0.055 0.021 0.0" rpy="0.656 0 0" /> <!-- Previous 0.656 0.3927 -->
+      <origin xyz="-0.055 0.021 0.0" rpy="0 0 0" /> <!-- Previous 0.656 0.3927 -->
       <axis xyz="1 0 0" />
       <limit velocity="6.5" effort="1000" lower="-3.14" upper="3.14" />
@@ -214,5 +214,5 @@
       <parent link="main_base"/>
       <child link="left_top_leg"/>
-      <origin xyz="0.101 0.021 0.0" rpy="0.656 0 0" />
+      <origin xyz="0.101 0.021 0.0" rpy="0 0 0" />
       <axis xyz="1 0 0" />
       <limit velocity="6.5" effort="1000" lower="-3.14" upper="3.14" />
@@ -222,5 +222,5 @@
       <parent link="right_top_leg"/>
       <child link="right_bottom_leg"/>
-      <origin xyz="-0.0 0.0 -0.1105" rpy="-1.67 0 0" /> <!-- Previous -1.67 -0.9547-->
+      <origin xyz="-0.0 0.0 -0.1105" rpy="0 0 0" /> <!-- Previous -1.67 -0.9547-->
       <axis xyz="1 0 0" />
       <limit velocity="6.5" effort="1000" lower="-3.14" upper="3.14" />
@@ -230,5 +230,5 @@
       <parent link="left_top_leg"/>
       <child link="left_bottom_leg"/>
-      <origin xyz="-0.0 0.0 -0.1105" rpy="-1.67 0 0" />
+      <origin xyz="-0.0 0.0 -0.1105" rpy="0 0 0" />
       <axis xyz="1 0 0" />
       <limit velocity="6.5" effort="1000" lower="-3.14" upper="3.14" />
@@ -270,8 +270,8 @@
       <type>transmission_interface/SimpleTransmission</type>
       <joint name="base2right_top_leg">
-          <hardwareInterface>hardware_interface/EffortJointInterface</hardwareInterface>
+          <hardwareInterface>hardware_interface/PositionJointInterface</hardwareInterface>
       </joint>
       <actuator name="motor_base2right_top_leg">
-        <hardwareInterface>hardware_interface/EffortJointInterface</hardwareInterface>
+        <hardwareInterface>hardware_interface/PositionJointInterface</hardwareInterface>
         <mechanicalReduction>1</mechanicalReduction>
       </actuator>
@@ -280,8 +280,8 @@
       <type>transmission_interface/SimpleTransmission</type>
       <joint name="base2left_top_leg">
-          <hardwareInterface>hardware_interface/EffortJointInterface</hardwareInterface>
+          <hardwareInterface>hardware_interface/PositionJointInterface</hardwareInterface>
       </joint>
       <actuator name="motor_base2left_top_leg">
-        <hardwareInterface>hardware_interface/EffortJointInterface</hardwareInterface>
+        <hardwareInterface>hardware_interface/PositionJointInterface</hardwareInterface>
         <mechanicalReduction>1</mechanicalReduction>
       </actuator>
@@ -290,8 +290,8 @@
       <type>transmission_interface/SimpleTransmission</type>
       <joint name="right_top_leg2bottom_leg">
-          <hardwareInterface>hardware_interface/EffortJointInterface</hardwareInterface>
+          <hardwareInterface>hardware_interface/PositionJointInterface</hardwareInterface>
       </joint>
       <actuator name="motor_right_top_leg2bottom_leg">
-        <hardwareInterface>hardware_interface/EffortJointInterface</hardwareInterface>
+        <hardwareInterface>hardware_interface/PositionJointInterface</hardwareInterface>
         <mechanicalReduction>1</mechanicalReduction>
       </actuator>
@@ -300,8 +300,8 @@
       <type>transmission_interface/SimpleTransmission</type>
       <joint name="left_top_leg2bottom_leg">
-          <hardwareInterface>hardware_interface/EffortJointInterface</hardwareInterface>
+          <hardwareInterface>hardware_interface/PositionJointInterface</hardwareInterface>
       </joint>
       <actuator name="motor_left_top_leg2bottom_leg">
-        <hardwareInterface>hardware_interface/EffortJointInterface</hardwareInterface>
+        <hardwareInterface>hardware_interface/PositionJointInterface</hardwareInterface>
         <mechanicalReduction>1</mechanicalReduction>
       </actuator>

Commit message: Fix controller issues

File: bbot_description/urdf/bbot.urdf.xacro (robot description, xacro)
@@ -426,5 +426,5 @@
       <sensor type="gpu_ray" name="lds_sensor">
         <pose>0 0 0 0 0 0</pose>
-        <visualize>true</visualize>
+        <visualize>false</visualize>
         <update_rate>40</update_rate>
         <ray>

File: bbot_description/urdf/ramp.urdf.xacro (robot description, xacro)
@@ -17,5 +17,5 @@
         <origin xyz="0.0 0.0 0.0" rpy="0 0 0" />
         <geometry>
-          <mesh filename="package://bbot_description/meshes/visual/Ramp.dae"  scale="1 1 1"/>
+          <mesh filename="package://bbot_description/meshes/visual/Ramp.dae"  scale="1 3 1"/>
         </geometry>
       </visual>
@@ -23,5 +23,5 @@
         <origin xyz="0.0 0.0 0.0" rpy="0 0 0" />
         <geometry>
-          <mesh filename="package://bbot_description/meshes/collision/Ramp.stl"  scale="1 1 1"/>
+          <mesh filename="package://bbot_description/meshes/collision/Ramp.stl"  scale="1 3 1"/>
         </geometry>
       </collision>

Commit message: correct K to pose C

File: bbot_description/urdf/bbot.urdf.xacro (robot description, xacro)
@@ -206,5 +206,5 @@
       <parent link="main_base"/>
       <child link="right_top_leg"/>
-      <origin xyz="-0.055 0.021 0.0" rpy="0 0 0" /> <!-- Previous 0.656 0.3927 -->
+      <origin xyz="-0.055 0.021 0.0" rpy="0.6545 0 0" /> <!-- Previous 0.656 0.3927 -->
       <axis xyz="1 0 0" />
       <limit velocity="6.5" effort="1000" lower="-3.14" upper="3.14" />
@@ -214,5 +214,5 @@
       <parent link="main_base"/>
       <child link="left_top_leg"/>
-      <origin xyz="0.101 0.021 0.0" rpy="0 0 0" />
+      <origin xyz="0.101 0.021 0.0" rpy="0.6545 0 0" />
       <axis xyz="1 0 0" />
       <limit velocity="6.5" effort="1000" lower="-3.14" upper="3.14" />
@@ -222,5 +222,5 @@
       <parent link="right_top_leg"/>
       <child link="right_bottom_leg"/>
-      <origin xyz="-0.0 0.0 -0.1105" rpy="0 0 0" /> <!-- Previous -1.67 -0.9547-->
+      <origin xyz="-0.0 0.0 -0.1105" rpy="-1.665 0 0" /> <!-- Previous -1.67 -0.9547-->
       <axis xyz="1 0 0" />
       <limit velocity="6.5" effort="1000" lower="-3.14" upper="3.14" />
@@ -230,5 +230,5 @@
       <parent link="left_top_leg"/>
       <child link="left_bottom_leg"/>
-      <origin xyz="-0.0 0.0 -0.1105" rpy="0 0 0" />
+      <origin xyz="-0.0 0.0 -0.1105" rpy="-1.665 0 0" />
       <axis xyz="1 0 0" />
       <limit velocity="6.5" effort="1000" lower="-3.14" upper="3.14" />

Commit message: add feature perception with bir_marker_localization and improve README

File: bbot_description/urdf/bbot.urdf.xacro (robot description, xacro)
@@ -410,10 +410,10 @@
     </gazebo>
     <!-- Optical frame -->
-      <!-- <link name="camera_optical_frame"/>
+      <link name="camera_optical_frame"/>
       <joint name="gazebo_optical_joint" type="fixed">
           <parent link="camera_frame_gazebo" />
           <child link="camera_optical_frame" />
           <origin xyz="0.0 0.0 0.0" rpy="-1.5708 0 -1.5708" />
-      </joint> -->
+      </joint>
   <!-- LiDAR -->
     <link name="lds_frame_gazebo"/>
