Commit message: Add navigation world

File: bbot_description/urdf/ramp.urdf.xacro (robot description, xacro)
@@ -17,5 +17,5 @@
         <origin xyz="0.0 0.0 0.0" rpy="0 0 0" />
         <geometry>
-          <mesh filename="package://bbot_description/meshes/visual/Ramp.dae"  scale="1 3 1"/>
+          <mesh filename="package://bbot_description/meshes/visual/Ramp.dae"  scale="1 9 1"/>
         </geometry>
       </visual>
